File: hardware/The_QwiicNES.brd (EAGLE design)
At the start: 57.1 x 40.6 mm, 92 parts, among them J1 Qwiic, J2 Qwiic, J6 AVR_SPI_PROG_3X2TESTPOINTS, U2 3.3V, U3 ATmega32U4, Y2 32MHz

Commit message: x01 initial order
Parts:
- removed C10: 1.0uF, SparkFun-Capacitors:0402-TIGHT
- removed C2, C4: 22pF, SparkFun-Capacitors:0402-TIGHT
- removed R15: 10k, SparkFun-Resistors:0402-TIGHT
- removed R20, R21: 22, SparkFun-Resistors:0402-TIGHT
- removed R22, R23: 2.2k, SparkFun-Resistors:0402-TIGHT
- removed Y2: 32MHz, SparkFun-Clocks:CRYSTAL-SMD-2.0X1.6MM
- added C11, C12, C9: 1.0uF, SparkFun-Capacitors:0603
- added J7: NES_CONTROLLER_PORT, NES:NES_CONTROLLER_PORT_7PIN_90
- added JP2: JUMPER-SMT_2_NC_TRACE_SILK, SparkFun-Jumpers:SMT-JUMPER_2_NC_TRACE_SILK
- added R11, R12: 22, SparkFun-Resistors:0603
- added R13, R16: 5.1k, SparkFun-Resistors:0603
- added R17: 2.2k, SparkFun-Resistors:0603
- added U$41: (no value), SparkFun-Aesthetics:QWIIC_5MM
- added Y1: 16MHz, SparkFun-Clocks:CRYSTAL-SMD-2.0X1.6MM
- C1, C3: value 0.1uF -> 22pF; device SparkFun-Capacitors:0402-TIGHT -> SparkFun-Capacitors:0603
- C5, C6: value 1.0uF -> 0.1uF; device SparkFun-Capacitors:0402-TIGHT -> SparkFun-Capacitors:0603
- J1, J2: value Qwiic -> QWIIC_RIGHT_ANGLE
- R1, R10, R2, R3, R4, R5, R6, R7, R8, R9: value 10k -> 1k
- R14: value 1k -> 10k; device SparkFun-Resistors:0402-TIGHT -> SparkFun-Resistors:0603
- R18: value 5.1k -> 2.2k; device SparkFun-Resistors:0402-TIGHT -> SparkFun-Resistors:0603
- R19: value 5.1k -> 1k; device SparkFun-Resistors:0402-TIGHT -> SparkFun-Resistors:0603
- U$2: value NES_CONTROLLER_PORT -> (none); device NES:NES_CONTROLLER_PORT_7PIN_90 -> SparkX:SPARKX-SMALL
- U$36: device SparkFun-Aesthetics:QWIIC_4MM -> output:#LED#0
- U$38: device SparkX:SPARKX-TINY -> SparkFun-Hardware:STAND-OFF-TIGHT
- moved R19 50.0 mm to (53.3, 30.5), turned to 180 degrees
- moved C6 32.1 mm to (34.7, 19.7), turned to 180 degrees
- moved U$38 30.2 mm to (54.6, 38.1)
- moved R18 29.5 mm to (34.3, 30.5), turned to 180 degrees
- moved R10 22.9 mm to (40.6, 15.2)
- moved U$36 19.3 mm to (51.7, 30.5), flipped to the bottom, turned to 270 degrees
- moved U$2 17.7 mm to (29.2, 22.1)
- moved C1 14.1 mm to (35.6, 34.3), turned to 270 degrees
- moved C3 9.64 mm to (40.6, 34.3), turned to 90 degrees
- moved R14 8.52 mm to (45.7, 31.8)
- moved C5 7.08 mm to (40.6, 19.1), turned to 90 degrees
- moved J6 6.88 mm to (47.0, 17.8), turned to 90 degrees
- moved U$34 5.09 mm to (45.7, 1.40)
- moved LED1 5.08 mm to (53.3, 31.8), turned to 180 degrees
- moved U$17 5.08 mm to (45.7, 1.78)
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Connections:
- removed net N$38: LED1.A, R14.1
- new net N$13: JP2.2, R19.1
- new net N$14: JP2.1, LED1.A
- net !RESET: now also R14.1; no longer R15.1
- net 3.3V: now also C11.1, C6.1, J3.2, J7.7, R19.2; no longer C10.2, C3.2, J3.4, R15.2, U$2.7
- net AREF: now also C5.1; no longer C1.2
- net A_LED: now also R6.2; no longer R7.2
- net B_LED: now also R7.2; no longer R8.2
- net D-_HV: now also R12.1; no longer R20.1
- net DN_LED: now also R1.2; no longer R2.2
- net DP_HV: now also R11.1; no longer R21.1
- net D_N: now also R12.2; no longer R20.2
- net D_P: now also R11.2; no longer R21.2
- net GND: now also C11.2, C12.2, C5.2, C6.2, C9.2, J7.1, R13.2, R16.2; no longer C10.1, C2.2, C4.2, C5.1, C6.1, R18.1, R19.1, U$2.1
- net LF_LED: now also R2.2; no longer R3.2
- net N$1: now also C3.2, Y1.1; no longer C4.1, Y2.1
- net N$10: now also R16.1; no longer R18.2
- net N$11: now also R7.1; no longer R8.1
- net N$12: now also R6.1; no longer R7.1
- net N$2: now also C1.2, Y1.3; no longer C2.1, Y2.3
- net N$21: now also R17.2; no longer R23.2
- net N$22: now also R18.2; no longer R22.2
- net N$23: now also R9.1; no longer R10.1
- net N$24: now also R8.1; no longer R9.1
- net N$3: now also R10.1; no longer R1.1
- net N$4: now also R1.1; no longer R2.1
- net N$5: now also R2.1; no longer R3.1
- net N$6: now also R3.1; no longer R4.1
- net N$7: now also R4.1; no longer R5.1
- net N$8: now also R5.1; no longer R6.1
- net N$9: now also R13.1; no longer R19.2
- net NES_CLK: now also J7.2; no longer U$2.2
- net NES_DATA: now also J7.4; no longer U$2.4
- net NES_LATCH: now also J7.3; no longer U$2.3
- net RT_LED: now also R3.2; no longer R4.2
- net SCL: now also J3.4, R17.1; no longer J3.3, R23.1
- net SDA: now also J3.3, R18.1; no longer J3.2, R22.1
- net SELECT_LED: now also R5.2; no longer R6.2
- net START_LED: now also R4.2; no longer R5.2
- net UCAP: now also C12.1; no longer C5.2
- net UP_LED: now also R10.2; no longer R1.2
- net V_USB: now also C9.1; no longer C6.2
- net ZAP_LIGHT: now also J7.6; no longer U$2.6
- net ZAP_LIGHT_LED: now also R9.2; no longer R10.2
- net ZAP_TRIGGER: now also J7.5; no longer U$2.5
- net ZAP_TRIG_LED: now also R8.2; no longer R9.2
Routing:
- net DO: track 6.74 -> 17.6 mm
- net DI: track 8.10 -> 18.8 mm, vias 0 -> 1
- net 3.3V: track 136.7 -> 129.0 mm, vias 6 -> 4
- net GND: track 16.9 -> 22.7 mm, vias 17 -> 16
- net SCK: track 10.2 -> 14.3 mm
- net N$14: track 0.00 -> 3.75 mm, vias 0 -> 1
- net N$13: track 0.00 -> 3.68 mm, vias 0 -> 1
- net V_USB: track 71.1 -> 74.6 mm
- net AREF: track 1.13 -> 4.30 mm
- net DP_HV: track 4.86 -> 8.03 mm
- net !RESET: track 24.4 -> 22.1 mm
- net SDA: track 55.8 -> 53.8 mm
- net N$10: track 2.81 -> 4.90 mm
- net SCL: track 55.0 -> 53.0 mm
- net D_N: track 41.4 -> 43.3 mm
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Other:
- board text added: "NPOOLE"
