File: hardware/The_QwiicNES.brd (EAGLE design)
At the start: 57.1 x 40.6 mm, 95 parts, among them J1 QWIIC_RIGHT_ANGLE, J2 QWIIC_RIGHT_ANGLE, J6 AVR_SPI_PROG_3X2TESTPOINTS, J7 NES_CONTROLLER_PORT, U2 3.3V, U3 ATmega32U4, Y1 16MHz

Commit message: reduced paste on main IC
Parts:
- U3: value ATmega32U4 -> 32U4; device SparkFun-IC-Microcontroller:QFN-44-NOPAD_1:1 -> SparkFun-IC-Microcontroller:QFN-44-NOPAD_1:1-LESS_PASTE
