File: hardware/The_QwiicNES.sch (EAGLE design)
At the start: 53 parts, among them J1 Qwiic, J2 Qwiic, J6 AVR_SPI_PROG_3X2TESTPOINTS, U2 3.3V, U3 ATmega32U4, Y2 32MHz

Commit message: x01 initial order
Parts:
- removed C10: 1.0uF, SparkFun-Capacitors:1.0UF-0402T-16V-10%
- removed C2, C4: 22pF, SparkFun-Capacitors:22PF-0402T-16V-10%
- removed R15: 10k, SparkFun-Resistors:10KOHM-0402T-1/16W-1%
- removed R20, R21: 22, SparkFun-Resistors:22OHM-0402T-1/16W-1%
- removed R22, R23: 2.2k, SparkFun-Resistors:2.2KOHM-0402T-1/16W-1%
- removed U$2: NES_CONTROLLER_PORT, NES:NES_CONTROLLER_PORT
- removed Y2: 32MHz, SparkFun-Clocks:CRYSTAL-32MHZ-SMD-2.0X1.6MM
- added C11, C12, C9: 1.0uF, SparkFun-Capacitors:1.0UF-0603-16V-10%
- added J7: NES_CONTROLLER_PORT, NES:NES_CONTROLLER_PORT
- added JP2: JUMPER-SMT_2_NC_TRACE_SILK, SparkFun-Jumpers:JUMPER-SMT_2_NC_TRACE_SILK
- added R11, R12: 22, SparkFun-Resistors:22OHM-0603-1/10W-1%
- added R13, R16: 5.1k, SparkFun-Resistors:5.1KOHM5.1KOHM-0603-1/10W-1%
- added R17: 2.2k, SparkFun-Resistors:2.2KOHM-0603-1/10W-1%
- added Y1: 16MHz, SparkFun-Clocks:CRYSTAL-16MHZSMD-2X1.6
- C1, C3: value 0.1uF -> 22pF; device SparkFun-Capacitors:0.1UF-0402T-16V-10% -> SparkFun-Capacitors:22PF-0603-50V-5%
- C5, C6: value 1.0uF -> 0.1uF; device SparkFun-Capacitors:1.0UF-0402T-16V-10% -> SparkFun-Capacitors:0.1UF-0603-25V-(+80/-20%)
- J1, J2: value Qwiic -> QWIIC_RIGHT_ANGLE
- R1, R10, R2, R3, R4, R5, R6, R7, R8, R9: value 10k -> 1k; device SparkFun-Resistors:10KOHM-0603-1/10W-1% -> SparkFun-Resistors:1KOHM-0603-1/10W-1%
- R14: value 1k -> 10k; device SparkFun-Resistors:1KOHM-0402T-1/16W-1% -> SparkFun-Resistors:10KOHM-0603-1/10W-1%
- R18: value 5.1k -> 2.2k; device SparkFun-Resistors:5.1KOHM-0402T-1/16W-1% -> SparkFun-Resistors:2.2KOHM-0603-1/10W-1%
- R19: value 5.1k -> 1k; device SparkFun-Resistors:5.1KOHM-0402T-1/16W-1% -> SparkFun-Resistors:1KOHM-0603-1/10W-1%
Connections:
- removed net N$38: LED1.A, R14.1
- new net N$13: JP2.2, R19.1
- new net N$14: JP2.1, LED1.A
- net !RESET: now also R14.1; no longer R15.1
- net 3.3V: now also C11.1, C6.1, J3.2, J7.VCC, R19.2; no longer C10.2, C3.2, J3.4, R15.2, U$2.VCC
- net AREF: now also C5.1; no longer C1.2
- net A_LED: now also R6.2; no longer R7.2
- net B_LED: now also R7.2; no longer R8.2
- net D-_HV: now also R12.1; no longer R20.1
- net DN_LED: now also R1.2; no longer R2.2
- net DP_HV: now also R11.1; no longer R21.1
- net D_N: now also R12.2; no longer R20.2
- net D_P: now also R11.2; no longer R21.2
- net GND: now also C11.2, C12.2, C5.2, C6.2, C9.2, J7.GND, R13.2, R16.2; no longer C10.1, C2.2, C4.2, C5.1, C6.1, R18.1, R19.1, U$2.GND
- net LF_LED: now also R2.2; no longer R3.2
- net N$1: now also C3.2, Y1.1; no longer C4.1, Y2.1
- net N$10: now also R16.1; no longer R18.2
- net N$11: now also R7.1; no longer R8.1
- net N$12: now also R6.1; no longer R7.1
- net N$2: now also C1.2, Y1.2; no longer C2.1, Y2.2
- net N$21: now also R17.2; no longer R23.2
- net N$22: now also R18.2; no longer R22.2
- net N$23: now also R9.1; no longer R10.1
- net N$24: now also R8.1; no longer R9.1
- net N$3: now also R10.1; no longer R1.1
- net N$4: now also R1.1; no longer R2.1
- net N$5: now also R2.1; no longer R3.1
- net N$6: now also R3.1; no longer R4.1
- net N$7: now also R4.1; no longer R5.1
- net N$8: now also R5.1; no longer R6.1
- net N$9: now also R13.1; no longer R19.2
- net NES_CLK: now also J7.CLOCK; no longer U$2.CLOCK
- net NES_DATA: now also J7.D1; no longer U$2.D1
- net NES_LATCH: now also J7.LATCH; no longer U$2.LATCH
- net RT_LED: now also R3.2; no longer R4.2
- net SCL: now also J3.4, R17.1; no longer J3.3, R23.1
- net SDA: now also J3.3, R18.1; no longer J3.2, R22.1
- net SELECT_LED: now also R5.2; no longer R6.2
- net START_LED: now also R4.2; no longer R5.2
- net UCAP: now also C12.1; no longer C5.2
- net UP_LED: now also R10.2; no longer R1.2
- net V_USB: now also C9.1; no longer C6.2
- net ZAP_LIGHT: now also J7.D3; no longer U$2.D3
- net ZAP_LIGHT_LED: now also R9.2; no longer R10.2
- net ZAP_TRIGGER: now also J7.D4; no longer U$2.D4
- net ZAP_TRIG_LED: now also R8.2; no longer R9.2
Other:
- moved on the sheet: C1, C3, C5, C6, C7, C8, D12, F1, LED1, R1, R10, R14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
