File: hardware/Production/The_QwiicNES-Panel.brd (EAGLE design)
At the start: 128.5 x 152.4 mm, 570 parts, among them J1 QWIIC_RIGHT_ANGLE, J11 QWIIC_RIGHT_ANGLE, J14 AVR_SPI_PROG_3X2TESTPOINTS, J15 NES_CONTROLLER_PORT, J16 QWIIC_RIGHT_ANGLE, J18 QWIIC_RIGHT_ANGLE, J2 QWIIC_RIGHT_ANGLE, J21 AVR_SPI_PROG_3X2TESTPOINTS, J22 NES_CONTROLLER_PORT, J23 QWIIC_RIGHT_ANGLE, J25 QWIIC_RIGHT_ANGLE, J28 AVR_SPI_PROG_3X2TESTPOINTS, J29 NES_CONTROLLER_PORT, J30 QWIIC_RIGHT_ANGLE, J32 QWIIC_RIGHT_ANGLE, J35 AVR_SPI_PROG_3X2TESTPOINTS, J36 NES_CONTROLLER_PORT, J37 QWIIC_RIGHT_ANGLE, J39 QWIIC_RIGHT_ANGLE, J42 AVR_SPI_PROG_3X2TESTPOINTS, J6 AVR_SPI_PROG_3X2TESTPOINTS, J7 NES_CONTROLLER_PORT, J8 NES_CONTROLLER_PORT, J9 QWIIC_RIGHT_ANGLE, U1 ATmega32U4, U10 3.3V, U11 ATmega32U4, U12 3.3V, U2 3.3V, U3 ATmega32U4, U4 3.3V, U5 ATmega32U4, U6 3.3V, U7 ATmega32U4, U8 3.3V, U9 ATmega32U4, Y1 16MHz, Y2 16MHz, Y3 16MHz, Y4 16MHz, Y5 16MHz, Y6 16MHz

Commit message: reduced paste on main IC
Parts:
- U1, U11, U3, U5, U7, U9: value ATmega32U4 -> 32U4; device SparkFun-IC-Microcontroller:QFN-44-NOPAD_1:1 -> SparkFun-IC-Microcontroller:QFN-44-NOPAD_1:1-LESS_PASTE
Changed lines of the file:
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@@
 <?xml version="1.0" encoding="utf-8"?>
 <!DOCTYPE eagle SYSTEM "eagle.dtd">
-<eagle version="9.5.2">
+<eagle version="9.6.2">
 <drawing>
 <settings>
-<setting alwaysvectorfont="yes"/>
+<setting alwaysvectorfont="no"/>
 <setting verticaltext="up"/>
 </settings>
@@
 <layer number="1" name="Top" color="4" fill="1" visible="yes" active="yes"/>
 <layer number="2" name="Route2" color="16" fill="1" visible="no" active="no"/>
-<layer number="3" name="Route3" color="17" fill="1" visible="no" active="no"/>
-<layer number="4" name="Route4" color="18" fill="1" visible="no" active="no"/>
-<layer number="5" name="Route5" color="19" fill="1" visible="no" active="no"/>
-<layer number="6" name="Route6" color="25" fill="1" visible="no" active="no"/>
-<layer number="7" name="Route7" color="26" fill="1" visible="no" active="no"/>
-<layer number="8" name="Route8" color="27" fill="1" visible="no" active="no"/>
-<layer number="9" name="Route9" color="28" fill="1" visible="no" active="no"/>
-<layer number="10" name="Route10" color="29" fill="1" visible="no" active="no"/>
-<layer number="11" name="Route11" color="30" fill="1" visible="no" active="no"/>
-<layer number="12" name="Route12" color="20" fill="1" visible="no" active="no"/>
-<layer number="13" name="Route13" color="21" fill="1" visible="no" active="no"/>
-<layer number="14" name="Route14" color="22" fill="1" visible="no" active="no"/>
 <layer number="15" name="Route15" color="23" fill="1" visible="no" active="no"/>
 <layer number="16" name="Bottom" color="1" fill="1" visible="yes" active="yes"/>
@@
 <vertex x="52.451" y="29.21"/>
 </polygon>
-<text x="28.575" y="-1.778" size="1.778" layer="20" font="vector" ratio="15" align="center">Route Out</text>
+<text x="28.575" y="-1.778" size="1.778" layer="20" ratio="15" align="center">Route Out</text>
 <wire x1="57.658" y1="0" x2="57.658" y2="40.64" width="0.254" layer="20"/>
 <wire x1="57.658" y1="40.64" x2="114.808" y2="40.64" width="0.254" layer="20"/>
@@
 <vertex x="110.109" y="29.21"/>
 </polygon>
-<text x="86.233" y="-1.778" size="1.778" layer="20" font="vector" ratio="15" align="center">Route Out</text>
+<text x="86.233" y="-1.778" size="1.778" layer="20" ratio="15" align="center">Route Out</text>
 <wire x1="0" y1="44.196" x2="0" y2="84.836" width="0.254" layer="20"/>
 <wire x1="0" y1="84.836" x2="57.15" y2="84.836" width="0.254" layer="20"/>
@@
 <vertex x="52.451" y="73.406"/>
 </polygon>
-<text x="28.575" y="42.418" size="1.778" layer="20" font="vector" ratio="15" align="center">Route Out</text>
+<text x="28.575" y="42.418" size="1.778" layer="20" ratio="15" align="center">Route Out</text>
 <wire x1="57.658" y1="44.196" x2="57.658" y2="84.836" width="0.254" layer="20"/>
 <wire x1="57.658" y1="84.836" x2="114.808" y2="84.836" width="0.254" layer="20"/>
@@
 <vertex x="110.109" y="73.406"/>
 </polygon>
-<text x="86.233" y="42.418" size="1.778" layer="20" font="vector" ratio="15" align="center">Route Out</text>
+<text x="86.233" y="42.418" size="1.778" layer="20" ratio="15" align="center">Route Out</text>
 <wire x1="0" y1="88.392" x2="0" y2="129.032" width="0.254" layer="20"/>
 <wire x1="0" y1="129.032" x2="57.15" y2="129.032" width="0.254" layer="20"/>
@@
 <vertex x="52.451" y="117.602"/>
 </polygon>
-<text x="28.575" y="86.614" size="1.778" layer="20" font="vector" ratio="15" align="center">Route Out</text>
-<text x="28.575" y="130.81" size="1.778" layer="20" font="vector" ratio="15" align="center">Route Out</text>
+<text x="28.575" y="86.614" size="1.778" layer="20" ratio="15" align="center">Route Out</text>
+<text x="28.575" y="130.81" size="1.778" layer="20" ratio="15" align="center">Route Out</text>
 <wire x1="57.658" y1="88.392" x2="57.658" y2="129.032" width="0.254" layer="20"/>
 <wire x1="57.658" y1="129.032" x2="114.808" y2="129.032" width="0.254" layer="20"/>
@@
 <vertex x="110.109" y="117.602"/>
 </polygon>
-<text x="86.233" y="86.614" size="1.778" layer="20" font="vector" ratio="15" align="center">Route Out</text>
-<text x="86.233" y="130.81" size="1.778" layer="20" font="vector" ratio="15" align="center">Route Out</text>
+<text x="86.233" y="86.614" size="1.778" layer="20" ratio="15" align="center">Route Out</text>
+<text x="86.233" y="130.81" size="1.778" layer="20" ratio="15" align="center">Route Out</text>
 <wire x1="-0.254" y1="-9.906" x2="-0.254" y2="142.494" width="0.381" layer="46"/>
-<text x="-0.254" y="144.78" size="1.778" layer="46" font="vector" ratio="15" align="center">v-score</text>
+<text x="-0.254" y="144.78" size="1.778" layer="46" ratio="15" align="center">v-score</text>
 <wire x1="57.404" y1="-9.906" x2="57.404" y2="142.494" width="0.381" layer="46"/>
-<text x="57.404" y="144.78" size="1.778" layer="46" font="vector" ratio="15" align="center">v-score</text>
+<text x="57.404" y="144.78" size="1.778" layer="46" ratio="15" align="center">v-score</text>
 <wire x1="115.062" y1="-9.906" x2="115.062" y2="142.494" width="0.381" layer="46"/>
-<text x="115.062" y="144.78" size="1.778" layer="46" font="vector" ratio="15" align="center">v-score</text>
+<text x="115.062" y="144.78" size="1.778" layer="46" ratio="15" align="center">v-score</text>
 <wire x1="-6.858" y1="-3.556" x2="121.666" y2="-3.556" width="0.254" layer="20"/>
 <wire x1="121.666" y1="-3.556" x2="121.666" y2="-9.906" width="0.254" layer="20"/>
@@
 <attribute name="VALUE" x="53.34" y="32.385" size="0.6096" layer="27" font="vector" ratio="20" rot="R180" align="top-center"/>
 </element>
-<element name="U3" library="SparkFun-IC-Microcontroller" package="QFN-44-NOPAD_1:1" value="ATmega32U4" x="38.1" y="25.4" smashed="yes" rot="R180">
+<element name="U3" library="SparkFun-IC-Microcontroller" package="QFN-44-NOPAD_1:1-LESS_PASTE" value="32U4" x="38.1" y="25.4" smashed="yes" rot="R180">
 <attribute name="NAME" x="38.1" y="20.955" size="0.6096" layer="25" font="vector" ratio="20" rot="R180" align="bottom-center"/>
 <attribute name="PROD_ID" value="IC-10828" x="57.15" y="-6.35" size="1.778" layer="27" rot="R180" display="off"/>
@@
 <attribute name="VALUE" x="110.998" y="32.385" size="0.6096" layer="27" font="vector" ratio="20" rot="R180" align="top-center"/>
 </element>
-<element name="U1" library="SparkFun-IC-Microcontroller" package="QFN-44-NOPAD_1:1" value="ATmega32U4" x="95.758" y="25.4" smashed="yes" rot="R180">
+<element name="U1" library="SparkFun-IC-Microcontroller" package="QFN-44-NOPAD_1:1-LESS_PASTE" value="32U4" x="95.758" y="25.4" smashed="yes" rot="R180">
 <attribute name="NAME" x="95.758" y="20.955" size="0.6096" layer="25" font="vector" ratio="20" rot="R180" align="bottom-center"/>
 <attribute name="PROD_ID" value="IC-10828" x="114.808" y="-6.35" size="1.778" layer="27" rot="R180" display="off"/>
@@
 <attribute name="VALUE" x="53.34" y="76.581" size="0.6096" layer="27" font="vector" ratio="20" rot="R180" align="top-center"/>
 </element>
-<element name="U5" library="SparkFun-IC-Microcontroller" package="QFN-44-NOPAD_1:1" value="ATmega32U4" x="38.1" y="69.596" smashed="yes" rot="R180">
+<element name="U5" library="SparkFun-IC-Microcontroller" package="QFN-44-NOPAD_1:1-LESS_PASTE" value="32U4" x="38.1" y="69.596" smashed="yes" rot="R180">
 <attribute name="NAME" x="38.1" y="65.151" size="0.6096" layer="25" font="vector" ratio="20" rot="R180" align="bottom-center"/>
 <attribute name="PROD_ID" value="IC-10828" x="57.15" y="37.846" size="1.778" layer="27" rot="R180" display="off"/>
@@
 <attribute name="VALUE" x="110.998" y="76.581" size="0.6096" layer="27" font="vector" ratio="20" rot="R180" align="top-center"/>
 </element>
-<element name="U7" library="SparkFun-IC-Microcontroller" package="QFN-44-NOPAD_1:1" value="ATmega32U4" x="95.758" y="69.596" smashed="yes" rot="R180">
+<element name="U7" library="SparkFun-IC-Microcontroller" package="QFN-44-NOPAD_1:1-LESS_PASTE" value="32U4" x="95.758" y="69.596" smashed="yes" rot="R180">
 <attribute name="NAME" x="95.758" y="65.151" size="0.6096" layer="25" font="vector" ratio="20" rot="R180" align="bottom-center"/>
 <attribute name="PROD_ID" value="IC-10828" x="114.808" y="37.846" size="1.778" layer="27" rot="R180" display="off"/>
@@
 <attribute name="VALUE" x="53.34" y="120.777" size="0.6096" layer="27" font="vector" ratio="20" rot="R180" align="top-center"/>
 </element>
-<element name="U9" library="SparkFun-IC-Microcontroller" package="QFN-44-NOPAD_1:1" value="ATmega32U4" x="38.1" y="113.792" smashed="yes" rot="R180">
+<element name="U9" library="SparkFun-IC-Microcontroller" package="QFN-44-NOPAD_1:1-LESS_PASTE" value="32U4" x="38.1" y="113.792" smashed="yes" rot="R180">
 <attribute name="NAME" x="38.1" y="109.347" size="0.6096" layer="25" font="vector" ratio="20" rot="R180" align="bottom-center"/>
 <attribute name="PROD_ID" value="IC-10828" x="57.15" y="82.042" size="1.778" layer="27" rot="R180" display="off"/>
@@
 <attribute name="VALUE" x="110.998" y="120.777" size="0.6096" layer="27" font="vector" ratio="20" rot="R180" align="top-center"/>
 </element>
-<element name="U11" library="SparkFun-IC-Microcontroller" package="QFN-44-NOPAD_1:1" value="ATmega32U4" x="95.758" y="113.792" smashed="yes" rot="R180">
+<element name="U11" library="SparkFun-IC-Microcontroller" package="QFN-44-NOPAD_1:1-LESS_PASTE" value="32U4" x="95.758" y="113.792" smashed="yes" rot="R180">
 <attribute name="NAME" x="95.758" y="109.347" size="0.6096" layer="25" font="vector" ratio="20" rot="R180" align="bottom-center"/>
 <attribute name="PROD_ID" value="IC-10828" x="114.808" y="82.042" size="1.778" layer="27" rot="R180" display="off"/>
